Commit message: Updates

File: gripkit_cr_plus_l_cc/gripkit_cr_plus_l_cc_description/urdf/gripkit_cr_plus_l_cc.xacro (robot description, xacro)
@@ -4,4 +4,6 @@
 <xacro:include filename="$(find gripkit_cr_plus_l_cc_description)/urdf/gripkit_cr_plus_l_cc.trans" />
 <xacro:include filename="$(find gripkit_cr_plus_l_cc_description)/urdf/gripkit_cr_plus_l_cc.gazebo" />
+<link name="world">
+</link>
 <link name="base_footprint">
 </link>
@@ -346,4 +348,9 @@
   </collision>
 </link>
+<joint name="world_joint" type="fixed">
+  <origin xyz="0 0 0" rpy="0 0 0"/>
+  <parent link="world"/>
+  <child link="base_footprint"/>
+</joint>
 <joint name="base_footprint_joint" type="fixed">
   <origin xyz="0 0 0" rpy="0 0 0"/>

File: gripkit_cr_plus_l_dd/gripkit_cr_plus_l_dd_description/urdf/gripkit_cr_plus_l_dd.xacro (robot description, xacro)
@@ -4,4 +4,6 @@
 <xacro:include filename="$(find gripkit_cr_plus_l_dd_description)/urdf/gripkit_cr_plus_l_dd.trans" />
 <xacro:include filename="$(find gripkit_cr_plus_l_dd_description)/urdf/gripkit_cr_plus_l_dd.gazebo" />
+<link name="world">
+</link>
 <link name="base_footprint">
 </link>
@@ -346,4 +348,9 @@
   </collision>
 </link>
+<joint name="world_joint" type="fixed">
+  <origin xyz="0 0 0" rpy="0 0 0"/>
+  <parent link="world"/>
+  <child link="base_footprint"/>
+</joint>
 <joint name="base_footprint_joint" type="fixed">
   <origin xyz="0 0 0" rpy="0 0 0"/>
