Commit message: Updates

File: kmr_iiwa_gripkit_cr_plus_l_description/urdf/kmr_iiwa_gripkit_cr_plus_l.xacro (robot description, xacro)
@@ -26,5 +26,5 @@
   <xacro:include filename="$(find kmp200_description)/urdf/kmp200.xacro" />
   <joint name="Rigid01" type="fixed">
-    <origin xyz="0.358053 -0.183769 0.701151" rpy="0 0 -1.5708"/>
+    <origin xyz="0.3633 -0.1842 0.7011" rpy="0 0 -1.5708"/>
     <parent link="base_link"/>
     <child link="link_0"/>

Commit message: Reconfigurable moveit

File: kmr_iiwa_gripkit_cr_plus_l_description/urdf/kmr_iiwa_gripkit_cr_plus_l.xacro (robot description, xacro)
@@ -9,4 +9,5 @@
   <plugin name="control" filename="libgazebo_ros_control.so"/>
 </gazebo>
+<xacro:arg name="controller_type" default="Effort"/>
 <xacro:property name="body_color" value="Gazebo/Silver" />
 <xacro:include filename="$(find iiwa7_description)/urdf/iiwa7.xacro" />
@@ -23,6 +24,12 @@
   <xacro:include filename="$(find gripkit_cr_plus_l_dd_description)/urdf/gripkit_cr_plus_l_dd.xacro" />
 </xacro:if>
+<link name="world"/>
 <xacro:if value="${mobile_base == 'kmp200'}">
   <xacro:include filename="$(find kmp200_description)/urdf/kmp200.xacro" />
+  <joint name="world_joint" type="fixed">
+    <origin xyz="0 0 0" rpy="0 0 0"/>
+    <parent link="world"/>
+    <child link="base_link"/>
+  </joint>
   <joint name="Rigid01" type="fixed">
     <origin xyz="0.3633 -0.1842 0.7011" rpy="0 0 -1.5708"/>
@@ -32,5 +39,4 @@
 </xacro:if>
 <xacro:if value="${mobile_base == 'None'}">
-  <link name="world"/>
   <joint name="world_joint" type="fixed">
     <origin xyz="0 0 0" rpy="0 0 0"/>
