Commit message: name changes

File: kmriiwa_description/urdf/kmriiwa.xacro (robot description, xacro)
@@ -1,13 +1,13 @@
 <?xml version="1.0" ?>
 <robot name="kmriiwa" xmlns:xacro="http://www.ros.org/wiki/xacro">
+<xacro:arg name="robot_name" default="kmriiwa" />
+<xacro:property name="robot_name" value="$(arg robot_name)" />
+<xacro:arg name="hardware_interface" default="Effort" />
 <xacro:arg name="ee_type" default="bb" />
 <xacro:property name="ee_type" value="$(arg ee_type)" />
-<xacro:arg name="mobile_base" default="kmp200" />
-<xacro:property name="mobile_base" value="$(arg mobile_base)" />
 <xacro:include filename="$(find kmriiwa_description)/urdf/materials.xacro" />
 <gazebo>
   <plugin name="control" filename="libgazebo_ros_control.so"/>
 </gazebo>
-<xacro:arg name="controller_type" default="Effort"/>
 <xacro:property name="body_color" value="Gazebo/Silver" />
 <xacro:include filename="$(find iiwa7_description)/urdf/iiwa7.xacro" />
@@ -25,5 +25,5 @@
 </xacro:if>
 <link name="world"/>
-<xacro:if value="${mobile_base == 'kmp200'}">
+<xacro:if value="${robot_name == 'kmriiwa'}">
   <xacro:include filename="$(find kmp200_description)/urdf/kmp200.xacro" />
   <joint name="world_joint" type="fixed">
@@ -38,5 +38,5 @@
   </joint>
 </xacro:if>
-<xacro:if value="${mobile_base == 'None'}">
+<xacro:if value="${robot_name == 'iiwa'}">
   <joint name="world_joint" type="fixed">
     <origin xyz="0 0 0" rpy="0 0 0"/>
