Commit message: Updates

File: iiwa7_description/urdf/iiwa7.xacro (robot description, xacro)
@@ -7,5 +7,5 @@
 <link name="base_footprint">
 </link>
-<link name="base_link">
+<link name="link_0">
   <inertial>
     <origin xyz="-0.012832431040764161 -4.5637556731516346e-08 0.07010426148644754" rpy="0 0 0"/>
@@ -16,5 +16,5 @@
     <origin xyz="0 0 0" rpy="0 0 0"/>
     <geometry>
-      <mesh filename="package://iiwa7_description/meshes/base_link.stl" scale="0.001 0.001 0.001"/>
+      <mesh filename="package://iiwa7_description/meshes/link_0.stl" scale="0.001 0.001 0.001"/>
     </geometry>
     <material name="silver"/>
@@ -23,5 +23,5 @@
     <origin xyz="0 0 0" rpy="0 0 0"/>
     <geometry>
-      <mesh filename="package://iiwa7_description/meshes/base_link.stl" scale="0.001 0.001 0.001"/>
+      <mesh filename="package://iiwa7_description/meshes/link_0.stl" scale="0.001 0.001 0.001"/>
     </geometry>
   </collision>
@@ -295,5 +295,5 @@
   <origin xyz="0 0 0" rpy="0 0 0"/>
   <parent link="base_footprint"/>
-  <child link="base_link"/>
+  <child link="link_0"/>
 </joint>
 <joint name="Rigid01" type="fixed">
@@ -329,5 +329,5 @@
 <joint name="Rev01" type="revolute">
   <origin xyz="0.0 0.0 0.1475" rpy="0 0 0"/>
-  <parent link="base_link"/>
+  <parent link="link_0"/>
   <child link="link_1"/>
   <axis xyz="0.0 0.0 1.0"/>

Commit message: name changes

File: iiwa7_description/urdf/iiwa7.xacro (robot description, xacro)
@@ -263,5 +263,5 @@
   </collision>
 </link>
-<link name="flange">
+<link name="link_7">
   <inertial>
     <origin xyz="4.659054144329294e-06 1.7291653306211654e-08 0.009981852938580671" rpy="0 0 0"/>
@@ -272,5 +272,5 @@
     <origin xyz="0.0 0.0002 -1.2314" rpy="0 0 0"/>
     <geometry>
-      <mesh filename="package://iiwa7_description/meshes/flange.stl" scale="0.001 0.001 0.001"/>
+      <mesh filename="package://iiwa7_description/meshes/link_7.stl" scale="0.001 0.001 0.001"/>
     </geometry>
     <material name="silver"/>
@@ -279,5 +279,5 @@
     <origin xyz="0.0 0.0002 -1.2314" rpy="0 0 0"/>
     <geometry>
-      <mesh filename="package://iiwa7_description/meshes/flange.stl" scale="0.001 0.001 0.001"/>
+      <mesh filename="package://iiwa7_description/meshes/link_7.stl" scale="0.001 0.001 0.001"/>
     </geometry>
   </collision>
@@ -285,30 +285,30 @@
 <joint name="Rigid03" type="fixed">
   <origin xyz="-5e-06 -0.050302 0.01703" rpy="0 0 0"/>
-  <parent link="flange"/>
+  <parent link="link_7"/>
   <child link="screw_1"/>
 </joint>
 <joint name="Rigid04" type="fixed">
   <origin xyz="-0.050305 -2e-06 0.01703" rpy="0 0 0"/>
-  <parent link="flange"/>
+  <parent link="link_7"/>
   <child link="screw_2"/>
 </joint>
 <joint name="Rigid05" type="fixed">
   <origin xyz="-5e-06 0.050298 0.01703" rpy="0 0 0"/>
-  <parent link="flange"/>
+  <parent link="link_7"/>
   <child link="screw_3"/>
 </joint>
 <joint name="Rigid06" type="fixed">
   <origin xyz="0.050295 -2e-06 0.01703" rpy="0 0 0"/>
-  <parent link="flange"/>
+  <parent link="link_7"/>
   <child link="screw_4"/>
 </joint>
 <joint name="Rigid07" type="fixed">
   <origin xyz="0.035567 -0.035567 0.0121" rpy="0 0 0"/>
-  <parent link="flange"/>
+  <parent link="link_7"/>
   <child link="screw_5"/>
 </joint>
 <joint name="Rigid08" type="fixed">
   <origin xyz="-0.035567 0.035567 0.0121" rpy="0 0 0"/>
-  <parent link="flange"/>
+  <parent link="link_7"/>
   <child link="screw_6"/>
 </joint>
@@ -358,5 +358,5 @@
   <origin xyz="0.0 0.0705 0.0909" rpy="0 0 0"/>
   <parent link="link_6"/>
-  <child link="flange"/>
+  <child link="link_7"/>
   <axis xyz="0.0 0.0 1.0"/>
   <limit upper="3.054326" lower="-3.054326" effort="100" velocity="100"/>

File: kmr_iiwa_gripkit_cr_plus_l_description/urdf/kmr_iiwa_gripkit_cr_plus_l.xacro (robot description, xacro)
@@ -48,5 +48,5 @@
   <joint name="Rigid09" type="fixed">
     <origin xyz="0 0 0.0351" rpy="0 0 0"/>
-    <parent link="flange"/>
+    <parent link="link_7"/>
     <child link="SF-ISO50-CRG200_Customer"/>
   </joint>

Commit message: Parameter tuning

File: iiwa7_description/urdf/iiwa7.xacro (robot description, xacro)
@@ -318,5 +318,5 @@
   <child link="link_1"/>
   <axis xyz="0.0 0.0 1.0"/>
-  <limit upper="2.96706" lower="-2.96706" effort="100" velocity="10"/>
+  <limit upper="2.96706" lower="-2.96706" effort="320" velocity="10"/>
 </joint>
 <joint name="Rev02" type="revolute">
@@ -325,5 +325,5 @@
   <child link="link_2"/>
   <axis xyz="0.0 1.0 0.0"/>
-  <limit upper="2.094395" lower="-2.094395" effort="100" velocity="10"/>
+  <limit upper="2.094395" lower="-2.094395" effort="320" velocity="10"/>
 </joint>
 <joint name="Rev03" type="revolute">
@@ -332,5 +332,5 @@
   <child link="link_3"/>
   <axis xyz="0.0 0.0 1.0"/>
-  <limit upper="2.96706" lower="-2.96706" effort="100" velocity="10"/>
+  <limit upper="2.96706" lower="-2.96706" effort="176" velocity="10"/>
 </joint>
 <joint name="Rev04" type="revolute">
@@ -339,5 +339,5 @@
   <child link="link_4"/>
   <axis xyz="0.0 -1.0 0.0"/>
-  <limit upper="2.094395" lower="-2.094395" effort="100" velocity="10"/>
+  <limit upper="2.094395" lower="-2.094395" effort="176" velocity="10"/>
 </joint>
 <joint name="Rev05" type="revolute">
@@ -346,5 +346,5 @@
   <child link="link_5"/>
   <axis xyz="0.0 0.0 1.0"/>
-  <limit upper="2.96706" lower="-2.96706" effort="100" velocity="10"/>
+  <limit upper="2.96706" lower="-2.96706" effort="110" velocity="10"/>
 </joint>
 <joint name="Rev06" type="revolute">
@@ -353,5 +353,5 @@
   <child link="link_6"/>
   <axis xyz="0.0 1.0 0.0"/>
-  <limit upper="2.094395" lower="-2.094395" effort="100" velocity="10"/>
+  <limit upper="2.094395" lower="-2.094395" effort="40" velocity="10"/>
 </joint>
 <joint name="Rev07" type="revolute">
@@ -360,5 +360,5 @@
   <child link="link_7"/>
   <axis xyz="0.0 0.0 1.0"/>
-  <limit upper="3.054326" lower="-3.054326" effort="100" velocity="10"/>
+  <limit upper="3.054326" lower="-3.054326" effort="40" velocity="10"/>
 </joint>
 </robot>
