Commit message: Parameter tuning

File: gripkit_cr_plus_l_ad_description/urdf/gripkit_cr_plus_l_ad.xacro (robot description, xacro)
@@ -413,5 +413,5 @@
   <child link="CRG200_base_jaw_1"/>
   <axis xyz="1.0 0.0 0.0"/>
-  <limit upper="0.021" lower="-0.021" effort="100" velocity="100"/>
+  <limit upper="0.021" lower="-0.021" effort="100" velocity="10"/>
 </joint>
 <joint name="Slider02" type="prismatic">
@@ -420,5 +420,5 @@
   <child link="CRG200_base_jaw_2"/>
   <axis xyz="1.0 0.0 0.0"/>
-  <limit upper="0.021" lower="-0.021" effort="100" velocity="100"/>
+  <limit upper="0.021" lower="-0.021" effort="100" velocity="10"/>
 </joint>
 <joint name="Rigid11" type="fixed">

File: gripkit_cr_plus_l_bb_description/urdf/gripkit_cr_plus_l_bb.xacro (robot description, xacro)
@@ -313,5 +313,5 @@
   <child link="CRG200_base_jaw_1"/>
   <axis xyz="1.0 0.0 0.0"/>
-  <limit upper="0.021" lower="-0.021" effort="100" velocity="100"/>
+  <limit upper="0.021" lower="-0.021" effort="100" velocity="10"/>
 </joint>
 <joint name="Slider02" type="prismatic">
@@ -320,5 +320,5 @@
   <child link="CRG200_base_jaw_2"/>
   <axis xyz="1.0 0.0 0.0"/>
-  <limit upper="0.021" lower="-0.021" effort="100" velocity="100"/>
+  <limit upper="0.021" lower="-0.021" effort="100" velocity="10"/>
 </joint>
 <joint name="Rigid11" type="fixed">

File: gripkit_cr_plus_l_cc_description/urdf/gripkit_cr_plus_l_cc.xacro (robot description, xacro)
@@ -353,5 +353,5 @@
   <child link="CRG200_base_jaw_1"/>
   <axis xyz="1.0 0.0 0.0"/>
-  <limit upper="0.021" lower="-0.021" effort="100" velocity="100"/>
+  <limit upper="0.021" lower="-0.021" effort="100" velocity="10"/>
 </joint>
 <joint name="Slider02" type="prismatic">
@@ -360,5 +360,5 @@
   <child link="CRG200_base_jaw_2"/>
   <axis xyz="1.0 0.0 0.0"/>
-  <limit upper="0.021" lower="-0.021" effort="100" velocity="100"/>
+  <limit upper="0.021" lower="-0.021" effort="100" velocity="10"/>
 </joint>
 <joint name="Rigid11" type="fixed">

File: gripkit_cr_plus_l_dd_description/urdf/gripkit_cr_plus_l_dd.xacro (robot description, xacro)
@@ -353,5 +353,5 @@
   <child link="CRG200_base_jaw_1"/>
   <axis xyz="1.0 0.0 0.0"/>
-  <limit upper="0.021" lower="-0.021" effort="100" velocity="100"/>
+  <limit upper="0.021" lower="-0.021" effort="100" velocity="10"/>
 </joint>
 <joint name="Slider02" type="prismatic">
@@ -360,5 +360,5 @@
   <child link="CRG200_base_jaw_2"/>
   <axis xyz="1.0 0.0 0.0"/>
-  <limit upper="0.021" lower="-0.021" effort="100" velocity="100"/>
+  <limit upper="0.021" lower="-0.021" effort="100" velocity="10"/>
 </joint>
 <joint name="Rigid11" type="fixed">

File: iiwa7_description/urdf/iiwa7.xacro (robot description, xacro)
@@ -318,5 +318,5 @@
   <child link="link_1"/>
   <axis xyz="0.0 0.0 1.0"/>
-  <limit upper="2.96706" lower="-2.96706" effort="100" velocity="100"/>
+  <limit upper="2.96706" lower="-2.96706" effort="100" velocity="10"/>
 </joint>
 <joint name="Rev02" type="revolute">
@@ -325,5 +325,5 @@
   <child link="link_2"/>
   <axis xyz="0.0 1.0 0.0"/>
-  <limit upper="2.094395" lower="-2.094395" effort="100" velocity="100"/>
+  <limit upper="2.094395" lower="-2.094395" effort="100" velocity="10"/>
 </joint>
 <joint name="Rev03" type="revolute">
@@ -332,5 +332,5 @@
   <child link="link_3"/>
   <axis xyz="0.0 0.0 1.0"/>
-  <limit upper="2.96706" lower="-2.96706" effort="100" velocity="100"/>
+  <limit upper="2.96706" lower="-2.96706" effort="100" velocity="10"/>
 </joint>
 <joint name="Rev04" type="revolute">
@@ -339,5 +339,5 @@
   <child link="link_4"/>
   <axis xyz="0.0 -1.0 0.0"/>
-  <limit upper="2.094395" lower="-2.094395" effort="100" velocity="100"/>
+  <limit upper="2.094395" lower="-2.094395" effort="100" velocity="10"/>
 </joint>
 <joint name="Rev05" type="revolute">
@@ -346,5 +346,5 @@
   <child link="link_5"/>
   <axis xyz="0.0 0.0 1.0"/>
-  <limit upper="2.96706" lower="-2.96706" effort="100" velocity="100"/>
+  <limit upper="2.96706" lower="-2.96706" effort="100" velocity="10"/>
 </joint>
 <joint name="Rev06" type="revolute">
@@ -353,5 +353,5 @@
   <child link="link_6"/>
   <axis xyz="0.0 1.0 0.0"/>
-  <limit upper="2.094395" lower="-2.094395" effort="100" velocity="100"/>
+  <limit upper="2.094395" lower="-2.094395" effort="100" velocity="10"/>
 </joint>
 <joint name="Rev07" type="revolute">
@@ -360,5 +360,5 @@
   <child link="link_7"/>
   <axis xyz="0.0 0.0 1.0"/>
-  <limit upper="3.054326" lower="-3.054326" effort="100" velocity="100"/>
+  <limit upper="3.054326" lower="-3.054326" effort="100" velocity="10"/>
 </joint>
 </robot>

Commit message: Updates parameters

File: gripkit_cr_plus_l_ad_description/urdf/gripkit_cr_plus_l_ad.xacro (robot description, xacro)
@@ -3,4 +3,6 @@
 <xacro:include filename="$(find gripkit_cr_plus_l_ad_description)/urdf/gripkit_cr_plus_l_ad.trans" />
 <xacro:include filename="$(find gripkit_cr_plus_l_ad_description)/urdf/gripkit_cr_plus_l_ad.gazebo" />
+<xacro:property name="max_velocity" value="10"/>
+<xacro:property name="max_effort" value="100"/>
 <link name="SF-ISO50-CRG200_Customer">
   <inertial>
@@ -413,5 +415,5 @@
   <child link="CRG200_base_jaw_1"/>
   <axis xyz="1.0 0.0 0.0"/>
-  <limit upper="0.021" lower="-0.021" effort="100" velocity="10"/>
+  <limit upper="0.021" lower="-0.021" effort="${max_effort}" velocity="${max_velocity}"/>
 </joint>
 <joint name="Slider02" type="prismatic">
@@ -420,5 +422,5 @@
   <child link="CRG200_base_jaw_2"/>
   <axis xyz="1.0 0.0 0.0"/>
-  <limit upper="0.021" lower="-0.021" effort="100" velocity="10"/>
+  <limit upper="0.021" lower="-0.021" effort="${max_effort}" velocity="${max_velocity}"/>
 </joint>
 <joint name="Rigid11" type="fixed">

File: gripkit_cr_plus_l_bb_description/urdf/gripkit_cr_plus_l_bb.xacro (robot description, xacro)
@@ -3,4 +3,6 @@
 <xacro:include filename="$(find gripkit_cr_plus_l_bb_description)/urdf/gripkit_cr_plus_l_bb.trans" />
 <xacro:include filename="$(find gripkit_cr_plus_l_bb_description)/urdf/gripkit_cr_plus_l_bb.gazebo" />
+<xacro:property name="max_velocity" value="10"/>
+<xacro:property name="max_effort" value="100"/>
 <link name="SF-ISO50-CRG200_Customer">
   <inertial>
@@ -313,5 +315,5 @@
   <child link="CRG200_base_jaw_1"/>
   <axis xyz="1.0 0.0 0.0"/>
-  <limit upper="0.021" lower="-0.021" effort="100" velocity="10"/>
+  <limit upper="0.021" lower="-0.021" effort="${max_effort}" velocity="${max_velocity}"/>
 </joint>
 <joint name="Slider02" type="prismatic">
@@ -320,5 +322,5 @@
   <child link="CRG200_base_jaw_2"/>
   <axis xyz="1.0 0.0 0.0"/>
-  <limit upper="0.021" lower="-0.021" effort="100" velocity="10"/>
+  <limit upper="0.021" lower="-0.021" effort="${max_effort}" velocity="${max_velocity}"/>
 </joint>
 <joint name="Rigid11" type="fixed">

File: gripkit_cr_plus_l_cc_description/urdf/gripkit_cr_plus_l_cc.xacro (robot description, xacro)
@@ -3,4 +3,6 @@
 <xacro:include filename="$(find gripkit_cr_plus_l_cc_description)/urdf/gripkit_cr_plus_l_cc.trans" />
 <xacro:include filename="$(find gripkit_cr_plus_l_cc_description)/urdf/gripkit_cr_plus_l_cc.gazebo" />
+<xacro:property name="max_velocity" value="10"/>
+<xacro:property name="max_effort" value="100"/>
 <link name="SF-ISO50-CRG200_Customer">
   <inertial>
@@ -353,5 +355,5 @@
   <child link="CRG200_base_jaw_1"/>
   <axis xyz="1.0 0.0 0.0"/>
-  <limit upper="0.021" lower="-0.021" effort="100" velocity="10"/>
+  <limit upper="0.021" lower="-0.021" effort="${max_effort}" velocity="${max_velocity}"/>
 </joint>
 <joint name="Slider02" type="prismatic">
@@ -360,5 +362,5 @@
   <child link="CRG200_base_jaw_2"/>
   <axis xyz="1.0 0.0 0.0"/>
-  <limit upper="0.021" lower="-0.021" effort="100" velocity="10"/>
+  <limit upper="0.021" lower="-0.021" effort="${max_effort}" velocity="${max_velocity}"/>
 </joint>
 <joint name="Rigid11" type="fixed">

File: gripkit_cr_plus_l_dd_description/urdf/gripkit_cr_plus_l_dd.xacro (robot description, xacro)
@@ -3,4 +3,6 @@
 <xacro:include filename="$(find gripkit_cr_plus_l_dd_description)/urdf/gripkit_cr_plus_l_dd.trans" />
 <xacro:include filename="$(find gripkit_cr_plus_l_dd_description)/urdf/gripkit_cr_plus_l_dd.gazebo" />
+<xacro:property name="max_velocity" value="10"/>
+<xacro:property name="max_effort" value="100"/>
 <link name="SF-ISO50-CRG200_Customer">
   <inertial>
@@ -353,5 +355,5 @@
   <child link="CRG200_base_jaw_1"/>
   <axis xyz="1.0 0.0 0.0"/>
-  <limit upper="0.021" lower="-0.021" effort="100" velocity="10"/>
+  <limit upper="0.021" lower="-0.021" effort="${max_effort}" velocity="${max_velocity}"/>
 </joint>
 <joint name="Slider02" type="prismatic">
@@ -360,5 +362,5 @@
   <child link="CRG200_base_jaw_2"/>
   <axis xyz="1.0 0.0 0.0"/>
-  <limit upper="0.021" lower="-0.021" effort="100" velocity="10"/>
+  <limit upper="0.021" lower="-0.021" effort="${max_effort}" velocity="${max_velocity}"/>
 </joint>
 <joint name="Rigid11" type="fixed">

File: iiwa7_description/urdf/iiwa7.xacro (robot description, xacro)
@@ -3,4 +3,7 @@
 <xacro:include filename="$(find iiwa7_description)/urdf/iiwa7.trans" />
 <xacro:include filename="$(find iiwa7_description)/urdf/iiwa7.gazebo" />
+<!-- <xacro:property name="safety_controller_k_pos" value="100" />
+<xacro:property name="safety_controller_k_vel" value="2" />  -->
+<xacro:property name="max_velocity" value="10"/>
 <link name="screw_1">
   <inertial>
@@ -318,5 +321,7 @@
   <child link="link_1"/>
   <axis xyz="0.0 0.0 1.0"/>
-  <limit upper="2.96706" lower="-2.96706" effort="320" velocity="10"/>
+  <limit upper="2.96706" lower="-2.96706" effort="320" velocity="${max_velocity}"/>
+  <!-- <safety_controller soft_upper_limit="2.93215" soft_lower_limit="-2.93215"
+                     k_position="${safety_controller_k_pos}" k_velocity="${safety_controller_k_vel}"/>  -->
 </joint>
 <joint name="Rev02" type="revolute">
@@ -325,5 +330,7 @@
   <child link="link_2"/>
   <axis xyz="0.0 1.0 0.0"/>
-  <limit upper="2.094395" lower="-2.094395" effort="320" velocity="10"/>
+  <limit upper="2.094395" lower="-2.094395" effort="320" velocity="${max_velocity}"/>
+  <!-- <safety_controller soft_upper_limit="2.05949" soft_lower_limit="-2.05949"
+                     k_position="${safety_controller_k_pos}" k_velocity="${safety_controller_k_vel}"/>  -->
 </joint>
 <joint name="Rev03" type="revolute">
@@ -332,5 +339,7 @@
   <child link="link_3"/>
   <axis xyz="0.0 0.0 1.0"/>
-  <limit upper="2.96706" lower="-2.96706" effort="176" velocity="10"/>
+  <limit upper="2.96706" lower="-2.96706" effort="176" velocity="${max_velocity}"/>
+  <!-- <safety_controller soft_upper_limit="2.93215" soft_lower_limit="-2.93215"
+                     k_position="${safety_controller_k_pos}" k_velocity="${safety_controller_k_vel}"/>  -->
 </joint>
 <joint name="Rev04" type="revolute">
@@ -339,5 +348,7 @@
   <child link="link_4"/>
   <axis xyz="0.0 -1.0 0.0"/>
-  <limit upper="2.094395" lower="-2.094395" effort="176" velocity="10"/>
+  <limit upper="2.094395" lower="-2.094395" effort="176" velocity="${max_velocity}"/>
+  <!-- <safety_controller soft_upper_limit="2.05949" soft_lower_limit="-2.05949"
+                     k_position="${safety_controller_k_pos}" k_velocity="${safety_controller_k_vel}"/>  -->
 </joint>
 <joint name="Rev05" type="revolute">
@@ -346,5 +357,7 @@
   <child link="link_5"/>
   <axis xyz="0.0 0.0 1.0"/>
-  <limit upper="2.96706" lower="-2.96706" effort="110" velocity="10"/>
+  <limit upper="2.96706" lower="-2.96706" effort="110" velocity="${max_velocity}"/>
+  <!-- <safety_controller soft_upper_limit="2.93215" soft_lower_limit="-2.93215"
+                     k_position="${safety_controller_k_pos}" k_velocity="${safety_controller_k_vel}"/>  -->
 </joint>
 <joint name="Rev06" type="revolute">
@@ -353,5 +366,7 @@
   <child link="link_6"/>
   <axis xyz="0.0 1.0 0.0"/>
-  <limit upper="2.094395" lower="-2.094395" effort="40" velocity="10"/>
+  <limit upper="2.094395" lower="-2.094395" effort="40" velocity="${max_velocity}"/>
+  <!-- <safety_controller soft_upper_limit="2.05949" soft_lower_limit="-2.05949"
+                     k_position="${safety_controller_k_pos}" k_velocity="${safety_controller_k_vel}"/>  -->
 </joint>
 <joint name="Rev07" type="revolute">
@@ -360,5 +375,7 @@
   <child link="link_7"/>
   <axis xyz="0.0 0.0 1.0"/>
-  <limit upper="3.054326" lower="-3.054326" effort="40" velocity="10"/>
+  <limit upper="3.054326" lower="-3.054326" effort="40" velocity="${max_velocity}"/>
+  <!-- <safety_controller soft_upper_limit="3.01942" soft_lower_limit="-3.01942"
+                     k_position="${safety_controller_k_pos}" k_velocity="${safety_controller_k_vel}"/>  -->
 </joint>
 </robot>
